File: PCB/Joulev2_RealTime.brd (EAGLE design)
At the start: 85.1 x 72 mm, 127 parts, among them IC2 LM340S-12, IC3 LM340S-12, J1 2-PIN_2MM-V, K1 692112030100, K2 692112030100, K3 692112030100, K4 692112030100, K5 692112030100, Q1 N_CH_MOSFET_FDLBL260N100, U1 ATMEGA328P_TQFP, U2 74VHC_MUXSO16, U3 RFM69CW, U4 TUSB8041, U5 ADP1706ARDZ-1.1-R7, U6 TPS2561DRCT, U7 TPS2561DRCT, U8 ATTINY441/841SSU/SSUR, U9 TXB0108PWR, X1 J12HEADER_(JOULE), X2 J13HEADER_(JOULE), X4 TRAXXAS-CON, Y1 16MHz, Y2 24MHz

Commit message: inital commit
Connections:
- removed net NSS_3P3V: U3.7
- new net NSS_3V3: U3.7, U8.6
- net MISO_3V3: now also U8.8
- net MOSI_3V3: now also U8.7
- net SCK_3V3: now also U8.9
Changed lines of the file:
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@@
 <?xml version="1.0" encoding="utf-8"?>
 <!DOCTYPE eagle SYSTEM "eagle.dtd">
-<eagle version="8.1.0">
+<eagle version="8.1.1">
 <drawing>
 <settings>
@@
 <signal name="SCK_3V3">
 <contactref element="U3" pad="6"/>
+<contactref element="U8" pad="9"/>
+<wire x1="80.745" y1="2.885" x2="81.395" y2="26.41" width="0" layer="19" extent="1-1"/>
 </signal>
 <signal name="MISO_3V3">
 <contactref element="U3" pad="8"/>
+<contactref element="U8" pad="8"/>
+<wire x1="82.745" y1="17.885" x2="82.665" y2="26.41" width="0" layer="19" extent="1-1"/>
 </signal>
 <signal name="MOSI_3V3">
 <contactref element="U3" pad="5"/>
-</signal>
-<signal name="NSS_3P3V">
-<contactref element="U3" pad="7"/>
+<contactref element="U8" pad="7"/>
+<wire x1="78.745" y1="2.885" x2="82.665" y2="21.21" width="0" layer="19" extent="1-1"/>
 </signal>
 <signal name="DIO0_3V3">
@@
 <wire x1="67.4644" y1="17.77" x2="78.855" y2="26.41" width="0" layer="19" extent="1-1"/>
 </signal>
+<signal name="NSS_3V3">
+<contactref element="U8" pad="6"/>
+<contactref element="U3" pad="7"/>
+<wire x1="82.745" y1="2.885" x2="81.395" y2="21.21" width="0" layer="19" extent="1-1"/>
+</signal>
 </signals>

Commit message: inital commit
Parts:
- moved C2 195.2 mm to (-99.1, 118.1), turned to 0 degrees
- moved D1 187.0 mm to (-91.4, 118.1), turned to 0 degrees
- moved JP5 177.1 mm to (-82.5, 97.8), turned to 0 degrees
- moved U2 174.2 mm to (-99.1, 90.2)
- moved C3 173.8 mm to (-102.9, 118.1), turned to 0 degrees
- moved R1 172.2 mm to (-102.9, 99.1), turned to 0 degrees
- moved R3 171.8 mm to (-94.0, 99.1), turned to 0 degrees
- moved JP6 168.2 mm to (-71.1, 90.2)
- moved JP4 167.6 mm to (-73.7, 97.8), turned to 0 degrees
- moved C55 165.5 mm to (-91.4, 114.3), turned to 0 degrees
- moved C52 165.4 mm to (-87.6, 114.3), turned to 0 degrees
- moved U3 163.4 mm to (-85.1, 33.0), turned to 0 degrees
- moved FB5 161.7 mm to (-96.5, 104.1), turned to 0 degrees
- moved R36 161.7 mm to (-64.8, 118.1)
- moved C4 158.8 mm to (-66.0, 104.1), turned to 0 degrees
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Routing:
- net GND: track 394.1 -> 0.00 mm, vias 9 -> 0
- net 3.3V: track 230.2 -> 0.00 mm, vias 6 -> 0
- net 5V: track 177.8 -> 0.00 mm, vias 6 -> 0
- net 1.1V: track 146.1 -> 0.00 mm, vias 7 -> 0
- net ESTOP_GATE: track 141.6 -> 0.00 mm, vias 2 -> 0
- net VCC: track 134.3 -> 0.00 mm, vias 6 -> 0
- net DN1_VBUS: track 109.3 -> 0.00 mm, vias 4 -> 0
- net N$12: track 104.9 -> 0.00 mm, vias 4 -> 0
- net ESTOP_5V: track 61.6 -> 0.00 mm, vias 1 -> 0
- net DN3_VBUS: track 47.3 -> 0.00 mm, vias 2 -> 0
- net USB_SSTXP_DN4: track 46.8 -> 0.00 mm, vias 4 -> 0
- net N$2: track 41.4 -> 0.00 mm, vias 2 -> 0
- net N$35: track 39.5 -> 0.00 mm, vias 2 -> 0
- net N$31: track 31.0 -> 0.00 mm, vias 2 -> 0
- net USB_SSRXP_DN1: track 30.4 -> 0.00 mm, vias 2 -> 0
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- removed copper zone on layer 16, net GND
Other:
- board size 85.1 x 72 mm -> 12.7 x 2.3 mm

Commit message: 05/01/2017
Parts:
- C10, C11, C12, C13, C14, C15, C16, C17, C18, C19, C20, C21, C22, C23, C24, C25, C26, C27, C28, C29, C30, C31, C32, C33, C34, C35, C36, C37, C38, C39, C40, C41, C42, C43, C44, C45, C46, C47, C48, C49, C5, C50, C51, C52, C55, C56, C6, C7, C8, C9: device SparkFun-Capacitors:0603 -> rcl:C0603
- R20, R21, R22, R23, R24, R25, R26, R27, R28, R29, R30, R31, R32, R33, R34, R35, R36, R37, R38, R39, R40, R41, R42: device SparkFun-Resistors:0603 -> rcl:R0603
- moved C56 171.3 mm to (36.4, 4.70), flipped to the bottom, turned to 180 degrees
- moved C52 164.5 mm to (36.4, 6.20), flipped to the bottom, turned to 180 degrees
- moved R22 160.8 mm to (23.7, 20.1), turned to 180 degrees
- moved FB4 159.0 mm to (31.3, 1.54), turned to 270 degrees
- moved C7 157.6 mm to (25.4, 22.1)
- moved FB3 155.3 mm to (32.8, 1.57), turned to 270 degrees
- moved C32 154.5 mm to (14.0, 14.1), flipped to the bottom, turned to 270 degrees
- moved R38 154.0 mm to (32.3, 5.11), flipped to the bottom
- moved C27 153.6 mm to (25.5, 6.63), turned to 270 degrees
- moved C31 153.1 mm to (16.1, 14.1), flipped to the bottom, turned to 90 degrees
- moved C49 152.5 mm to (32.3, 7.20), flipped to the bottom, turned to 180 degrees
- moved C26 152.4 mm to (27.6, 6.57), turned to 270 degrees
- moved C30 152.0 mm to (18.2, 13.8), flipped to the bottom, turned to 90 degrees
- moved C29 151.6 mm to (9.87, 1.25), flipped to the bottom, turned to 90 degrees
- moved FB5 150.7 mm to (23.0, 12.4), flipped to the bottom, turned to 180 degrees
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Connections:
- removed net N$45: C56.1, C58.1, U7.8_1, U7.8_2
- net +3V3_HUB: now also U4.16, U4.34, U4.52, U4.63
- net DN4_VBUS: now also C56.1, C58.1, U7.8_1, U7.8_2
- net GND: now also K4.7, K5.7; no longer U4.16, U4.34, U4.52, U4.63
- net N$38: now also K3.1
Routing:
- net GND: track 0.00 -> 91.6 mm, vias 0 -> 29
- net USBA_USB3_1_RX_DN: track 0.00 -> 37.5 mm, vias 0 -> 2
- net USBA_USB2_1_DP: track 0.00 -> 36.6 mm
- net USBA_USB3_1_RX_DP: track 0.00 -> 36.3 mm, vias 0 -> 2
- net USBA_USB2_1_DN: track 0.00 -> 33.9 mm
- net N$38: track 0.00 -> 33.6 mm, vias 0 -> 1
- net Y: track 0.00 -> 28.3 mm, vias 0 -> 2
- net X: track 0.00 -> 26.2 mm
- net N$40: track 0.00 -> 25.9 mm, vias 0 -> 1
- net USB_SSRXM_DN1: track 0.00 -> 21.8 mm, vias 0 -> 2
- net 1.1V: track 0.00 -> 21.1 mm, vias 0 -> 4
- net USB_SSRXP_DN1: track 0.00 -> 17.7 mm, vias 0 -> 2
- net USB_SSRXM_DN3: track 0.00 -> 17.3 mm, vias 0 -> 2
- net N$35: track 0.00 -> 16.8 mm, vias 0 -> 1
- net USB_DP_DN1: track 0.00 -> 14.4 mm
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- added copper zone on layer 2, net +3V3_HUB
- added copper zone on layer 2, net 3.3V
- added copper zone on layer 3, net GND
Other:
- board size 12.7 x 2.3 mm -> 85.2 x 72.5 mm

Commit message: .
Parts:
- moved R27 3.78 mm to (27.6, 16.4)
- moved R38 3.60 mm to (28.7, 4.39), turned to 180 degrees
- moved C56 2.46 mm to (37.0, 7.08)
- moved R32 1.65 mm to (26.1, 14.1), turned to 180 degrees
- moved R25 1.50 mm to (24.5, 16.4)
- moved C52 1.40 mm to (37.0, 4.95)
- moved R33 0.71 mm to (26.1, 11.6)
- moved C54 0.62 mm to (37.8, 2.72)
- moved C58 0.62 mm to (37.8, 9.47)
- moved FB3 0.50 mm to (33.3, 1.57)
Routing:
- net OVERCUR3Z: track 0.00 -> 24.0 mm
- net OVERCUR4Z: track 0.00 -> 18.8 mm, vias 0 -> 2
- net DN4_VBUS: track 2.28 -> 13.7 mm, vias 0 -> 1
- net GND: track 91.6 -> 96.4 mm, vias 29 -> 32
- net N$22: track 2.40 -> 6.68 mm
- net DN3_VBUS: track 5.78 -> 8.72 mm
- net 3.3V: track 6.73 -> 5.18 mm, vias 3 -> 2
- net PWRCTL2_BATEN2: track 4.44 -> 5.39 mm
- net +5V: track 2.71 -> 3.50 mm
- net PWRCTL1_BATEN1: track 4.57 -> 5.10 mm

Commit message: cinco de mayo
Parts:
- added C62: 4.7uF, rcl:C0603
- added C63: 1.0uF, rcl:C0603
- C20, C21, C22, C23, C24, C25, C26, C27, C8, C9: device rcl:C0603 -> rcl:C0402
- moved R42 159.2 mm to (27.6, 8.26), flipped to the bottom, turned to 270 degrees
- moved R40 153.9 mm to (30.4, 10.9)
- moved C55 127.4 mm to (14.9, 44.2), flipped to the bottom, turned to 90 degrees
- moved C51 125.2 mm to (15.1, 37.4), flipped to the bottom, turned to 90 degrees
- moved C42 124.0 mm to (27.4, 17.1), turned to 180 degrees
- moved C43 123.7 mm to (29.8, 22.7)
- moved C34 105.6 mm to (33.5, 22.7), turned to 180 degrees
- moved ENCODER 11.4 mm to (-30.5, 97.8)
- moved IMU 11.4 mm to (-19.1, 97.8)
- moved U5 8.25 mm to (33.1, 18.9), turned to 90 degrees
- moved C48 2.19 mm to (4.55, 32.1), turned to 90 degrees
- moved R37 1.51 mm to (5.42, 36.5)
- moved C32 1.37 mm to (15.3, 14.6)
- moved C31 0.90 mm to (16.9, 13.6)
- moved C38 0.50 mm to (20.2, 18.9)
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Connections:
- net 3.3V: now also C63.1, IMU.2; no longer ENCODER.2
- net 5V: now also C62.1, ENCODER.1; no longer IMU.1
- net ACHANNEL_5V: now also ENCODER.2; no longer IMU.2
- net BCHANNEL_5V: now also ENCODER.4; no longer IMU.4
- net GND: now also C62.2, C63.2, ENCODER.3, IMU.1, U3.13; no longer ENCODER.1, IMU.3
- net I2C0_SCL: now also IMU.4; no longer ENCODER.4
- net I2C0_SDA: now also IMU.3; no longer ENCODER.3
- net N$26: now also U4.26; no longer U4.27
- net N$27: now also U4.27; no longer U4.26
- net N$28: now also U4.19; no longer U4.20
- net N$29: now also U4.20; no longer U4.19
- net N$30: now also U4.11; no longer U4.12
- net N$31: now also U4.12; no longer U4.11
- net N$32: now also U4.3; no longer U4.4
- net N$33: now also U4.4; no longer U4.3
Routing:
- net 1.1V: track 21.1 -> 77.7 mm, vias 4 -> 8
- net GND: track 96.4 -> 127.5 mm, vias 32 -> 55
- net DN2_VBUS: track 0.00 -> 20.1 mm, vias 0 -> 2
- net 3.3V: track 5.18 -> 22.1 mm, vias 2 -> 9
- net DN1_VBUS: track 0.00 -> 15.8 mm, vias 0 -> 1
- net PWRCTL1_BATEN1: track 5.10 -> 19.9 mm, vias 1 -> 3
- net N$27: track 13.3 -> 0.00 mm
- net PWRCTL2_BATEN2: track 5.39 -> 17.9 mm, vias 1 -> 3
- net N$26: track 11.3 -> 0.00 mm, vias 2 -> 0
- net +3V3_HUB: track 9.66 -> 20.2 mm, vias 3 -> 8
- net +5V: track 3.50 -> 8.83 mm, vias 1 -> 2
- net ILIM1: track 0.00 -> 4.30 mm, vias 0 -> 1
- net N$28: track 8.57 -> 6.17 mm
- net N$36: track 0.00 -> 2.10 mm
- net VBUS_HUB: track 0.00 -> 2.08 mm
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- added copper zone on layer 3, net +3V3_HUB
- added copper zone on layer 3, net 3.3V
- added copper zone on layer 2, net GND
- removed copper zone on layer 2, net +3V3_HUB
- removed copper zone on layer 2, net 3.3V
- removed copper zone on layer 3, net GND
