File: PCB/Joulev2_RealTime.sch (EAGLE design)
At the start: 112 parts, among them IC2 LM340S-12, IC3 LM340S-12, J1 2-PIN_2MM-V, J2 USB_A_SMT_FEMALE, J3 USB_A_SMT_FEMALE, J4 USB_A_SMT_FEMALE, J5 USB_A_SMT_FEMALE, J6 USB_A_SMT_FEMALE, Q1 N_CH_MOSFET_FDLBL260N100, U1 ATMEGA328P_TQFP, U2 74VHC_MUXSO16, U3 RFM69CW, U5 TPS2561DRCT, U6 TPS2561DRCT, U8 ATTINY441/841SSU/SSUR, U9 TXB0108PWR, X1 J12HEADER_(JOULE), X2 J13HEADER_(JOULE), X4 TRAXXAS-CON, Y1 16MHz, Y2 24MHz

Commit message: Revert "Merge remote-tracking branch 'origin/USB2.0' into Joule-Breakout"
This reverts commit 2839ac94d3ec3073ea43a796fe64a609bf76dc33, reversing
changes made to d49a66ea7caaff2f058e7b4f2c8019333170ecc5.
Parts:
- removed FB6: 220@100MHz, SparkFun-Coils:FERRITE_BEAD-0603
- removed J2, J3, J4, J5, J6: USB_A_SMT_FEMALE, SparkFun-Connectors:USB_A_SMT_FEMALE
- removed R10, R11, R12, R8, R9: 1M, rcl:R-US_R0603
- removed R13, R14, R15, R16, R4, R5: 4.7k, rcl:R-US_R0603
- removed R17: 25.5k, rcl:R-US_R0603
- removed R18, R19, R7: 10k, rcl:R-US_R0603
- removed R6: 90.9k, rcl:R-US_R0603
- removed U$1: TUSB4041, Roboracing:TUSB4041
- added C44, C45, C46, C47, C48, C49, C51, C52, C55, C56: 0.1uF, SparkFun-Capacitors:0.1UF-0603-25V-(+80/-20%)
- added C50: 10uF, SparkFun-Capacitors:10UF-0603-6.3V-20%
- added C53, C54, C57, C58: 150uF, SparkFun-Capacitors:100UF-POLAR-RADIAL-2.5MM-25V-20%
- added K1, K2, K3, K4, K5: 692112030100, Roboracing:692112030100
- added R27, R29, R32, R33, R34, R35: 4.7k, SparkFun-Resistors:4.7KOHM-0603-1/10W-1%
- added R28: 9.53k, SparkFun-Resistors:9.76KOHM-0603-1/10W-1%
- added R30, R31, R36: 1M, SparkFun-Resistors:1MOHM-0603-1/4W-5%
- added R37, R38: 25.5k, SparkFun-Resistors:26.7KOHM0603-1/10W-1%
- added R39, R40, R41, R42: 10k, SparkFun-Resistors:10KOHM-0603-1/10W-1%
- added U4: TUSB8041, Roboracing:TUSB8041
- added U7: TPS2561DRCT, Roboracing:TPS2561DRCT
- C10, C16, C19, C33, C5: value 0.1uF -> 1nF; device rcl:C-USC0603 -> SparkFun-Capacitors:1.0NF/1000PF-0603-50V-10%
- C11: value 1nF -> 1.0uF; device rcl:C-USC0603 -> SparkFun-Capacitors:1.0UF-0603-16V-10%
- C12, C13, C18, C22, C23, C26, C27, C31, C32, C35, C36, C37, C39, C40, C41, C9: device rcl:C-USC0603 -> SparkFun-Capacitors:0.1UF-0603-25V-(+80/-20%)
- C14: value 1nF -> 18pF; device rcl:C-USC0603 -> SparkFun-Capacitors:18PF-0603-50V-5%
- C15: value 0.1uF -> 18pF; device rcl:C-USC0603 -> SparkFun-Capacitors:18PF-0603-50V-5%
- C17, C8: value 1nF -> 0.1uF; device rcl:C-USC0603 -> SparkFun-Capacitors:0.1UF-0603-25V-(+80/-20%)
- C20, C21, C24, C25: value 150uF -> 0.1uF; device rcl:CPOL-USE3.5-8 -> SparkFun-Capacitors:0.1UF-0603-25V-(+80/-20%)
- C28: value (none) -> 0.1uF; device rcl:C-USC0603 -> SparkFun-Capacitors:0.1UF-0603-25V-(+80/-20%)
- C29: value 18pF -> 0.1uF; device rcl:C-USC0603 -> SparkFun-Capacitors:0.1UF-0603-25V-(+80/-20%)
- C30: value 18pF -> 10uF; device rcl:C-USC0603 -> SparkFun-Capacitors:10UF-0603-6.3V-20%
- C34: value 0.1uF -> 4.7uF; device rcl:C-USC0603 -> SparkFun-Capacitors:4.7UF0603
- C38: value 10uF -> 0.1uF; device rcl:C-USC0603 -> SparkFun-Capacitors:0.1UF-0603-25V-(+80/-20%)
- C42: value 0.1uF -> 10nF; device rcl:C-USC0603 -> SparkFun-Capacitors:10NF-0603-50V-10%
- C43: value 10uF -> 4.7uF; device rcl:C-USC0603 -> SparkFun-Capacitors:4.7UF0603
- C6: value 1.0nF -> 0.1uF; device rcl:C-USC0603 -> SparkFun-Capacitors:0.1UF-0603-25V-(+80/-20%)
- C7: device rcl:C-USC0603 -> SparkFun-Capacitors:10UF-0603-6.3V-20%
- FB4: value 220@100MHz -> 220@100Mhz
- R20: value 25.5k -> 1M; device rcl:R-US_R0603 -> SparkFun-Resistors:1MOHM-0603-1/4W-5%
- R21: value 10k -> 1M; device rcl:R-US_R0603 -> SparkFun-Resistors:1MOHM-0603-1/4W-5%
- R22: value 10k -> 90.9k; device rcl:R-US_R0603 -> SparkFun-Resistors:100KOHM-0603-1/10W-1%
- R23: value 9.53k -> 10k; device rcl:R-US_R0603 -> SparkFun-Resistors:10KOHM-0603-1/10W-1%
- R24, R25: device rcl:R-US_R0603 -> SparkFun-Resistors:4.7KOHM-0603-1/10W-1%
- R26: device rcl:R-US_R0603 -> SparkFun-Resistors:1MOHM-0603-1/4W-5%
- U5: value TPS2561DRCT -> ADP1706ARDZ-1.1-R7; device Roboracing:TPS2561DRCT -> Roboracing:ADP1706ARDZ-1.1-R7
Connections:
- removed net +3V3: FB5.2, FB6.2, R18.2, R19.2, R21.2, R22.2
- removed net N$14: R5.2, U$1G$4.GANGED/SMBA2/HS_UP
- removed net N$15: R6.2, R7.2, U$1G$4.USB_VBUS
- removed net N$16: C7.1, J6.VBUS, R6.1
- removed net N$17: C13.1, FB2.2, J3.VBUS
- removed net N$19: J6.D-, U$1G$4.USB_DM_UP
- removed net N$21: J6.D+, U$1G$4.USB_DP_UP
- removed net N$34: C31.1, C32.1, C33.1, C34.1, C35.1, C36.1, C37.1, C38.1, FB5.1, U$1G$3.VDD1, U$1G$3.VDD2, U$1G$3.VDD3, U$1G$3.VDD4, U$1G$3.VDD5, U$1G$3.VDD6, U$1G$3.VDD7
- removed net N$37: C8.1, C9.1, J2.SHIELD, R10.2
- removed net PWRCTL1: R13.1, U$1G$1.PWRCTL1/BATEN1, U6.EN1
- removed net PWRCTL2: R14.1, U6.EN2
- removed net PWRCTL3: R15.1, U5.EN1
- removed net PWRCTL4: R16.1, U5.EN2
- new net +3V3_HUB: C44.1, C45.1, C46.1, C47.1, C50.1, FB5.1
- new net 1.1V: C30.1, C31.1, C32.1, C35.1, C38.1, C39.1, C40.1, C41.1, C43.1, U4G$2.VDD1, U4G$2.VDD2, U4G$2.VDD3, U4G$2.VDD4, U4G$2.VDD5, U4G$2.VDD6, U4G$2.VDD7, U4G$2.VDD8, U5.OUT, U5.OUT2, U5.SENSE
- new net GRST#: C11.1, U4G$1.GRST#
- new net ILIM1: R37.2, U6.ILIM
- new net ILIM2: R38.2, U7.ILIM
- new net N$40: C28.1, FB3.2, K4.VBUS
- new net N$45: C56.1, C58.+, U7.OUT2
- new net N$73: C36.1, FB4.2, K5.VBUS
- new net PWRCTL1_BATEN1: R32.1, U4G$1.PWRCTL1/BATEN1, U6.EN1
- new net PWRCTL2_BATEN2: R33.1, U4G$1.PWRCTL2/BATEN2, U6.EN2
- new net PWRCTL3_BATEN3: R34.1, U4G$1.PWRCTL3/BATEN3, U7.EN1
- new net PWRCTL4_BATEN4: R35.1, U4G$1.PWRCTL4/BATEN4, U7.EN2
- new net USBA_USB2_1_DN: K1.D-, U4G$1.USB_DM_UP
- new net USBA_USB2_1_DP: K1.D+, U4G$1.USB_DP_UP
- new net USBA_USB3_1_RX_DN: K1.STDA_SSRX-, U4G$1.USB_SSRXM_UP
- new net USBA_USB3_1_RX_DP: K1.STDA_SSRX+, U4G$1.USB_SSRXP_UP
- new net USBA_USB3_1_TX_DN: C9.1, K1.STDA_SSTX-
- new net USBA_USB3_1_TX_DP: C8.1, K1.STDA_SSTX+
- new net USB_SSRXM_DN1: K2.STDA_SSRX-, U4G$1.USB_SSRXM_DN1
- new net USB_SSRXM_DN2: K3.STDA_SSRX-, U4G$1.USB_SSRXM_DN2
- new net USB_SSRXM_DN3: K4.STDA_SSRX-, U4G$1.USB_SSRXM_DN3
- new net USB_SSRXM_DN4: K5.STDA_SSRX-, U4G$1.USB_SSRXM_DN4
- new net USB_SSRXP_DN1: K2.STDA_SSRX+, U4G$1.USB_SSRXP_DN1
- new net USB_SSRXP_DN2: K3.STDA_SSRX+, U4G$1.USB_SSRXP_DN2
- new net USB_SSRXP_DN3: K4.STDA_SSRX+, U4G$1.USB_SSRXP_DN3
- new net USB_SSRXP_DN4: K5.STDA_SSRX+, U4G$1.USB_SSRXP_DN4
- new net USB_SSTXM_DN1: C21.2, K2.STDA_SSTX-
- new net USB_SSTXM_DN2: C23.2, K3.STDA_SSTX-
- new net USB_SSTXM_DN3: C25.2, K4.STDA_SSTX-
- new net USB_SSTXM_DN4: C27.2, K5.STDA_SSTX-
- new net USB_SSTXP_DN1: C20.2, K2.STDA_SSTX+
- new net USB_SSTXP_DN2: C22.2, K3.STDA_SSTX+
- new net USB_SSTXP_DN3: C24.2, K4.STDA_SSTX+
- new net USB_SSTXP_DN4: C26.2, K5.STDA_SSTX+
- new net VBUS_HUB: C7.1, K1.VBUS, R22.1
- new net X: C8.2, U4G$1.USB_SSTXP_UP
- new net XI: C15.2, R26.2, U4G$1.XI, Y2.2
- new net XO: C14.2, R26.1, U4G$1.XO, Y2.1
- new net Y: C9.2, U4G$1.USB_SSTXM_UP
- net +5V: now also C48.1, C49.1, U7.IN, U7.IN2; no longer U5.IN, U5.IN2
- net 3.3V: now also C34.1, FB5.2, R32.2, R33.2, R34.2, R35.2, R39.2, R40.2, R41.2, R42.2, U5.EN, U5.IN, U5.IN2; no longer R13.2, R14.2, R15.2, R16.2
- net DN1_VBUS: now also C51.1, C53.+; no longer C24.+, C27.1
- net DN2_VBUS: now also C55.1, C57.+; no longer C25.+, C26.1
- net DN3_VBUS: now also C52.1, C54.+, U7.OUT1; no longer C20.+, C23.1, U5.OUT1
- net DN4_VBUS: no longer C21.+, C22.1, U5.OUT2
- net GND: now also C10.1, C13.1, C14.1, C15.1, C16.1, C18.1, C19.1, C29.1, C33.1, C37.1, C44.2, C45.2, C46.2, C47.2, C48.2, C49.2, C5.1, C50.2, C51.2, C52.2, C53.-, C54.-, C55.2, C56.2, C57.-, C58.-, C6.1, K1.GND, K1.GND_DRAIN, K2.GND, K2.GND_DRAIN, K3.GND, K3.GND_DRAIN, K4.GND, K5.GND, R20.2, R21.1, R21.2, R27.1, R28.1, R29.1, R30.1, R30.2, R31.1, R31.2, R36.1, R36.2, R37.1, R38.1, U4G$2.PAD, U4G$2.VDD33_1, U4G$2.VDD33_2, U4G$2.VDD33_3, U4G$2.VDD33_4, U7.GND, U7.PAD; no longer C14.2, C15.2, C20.-, C21.-, C22.2, C23.2, C24.-, C25.-, C26.2, C27.2, C8.2, C9.2, J2.GND, J3.GND, J4.GND, J5.GND, J6.GND, R10.1, R11.1, R12.1, R17.1, R4.1, R5.1, R7.1, R8.1, R9.1, U$1G$3.THERMAL_PAD, U5.PAD
- net N$18: now also R29.2, U4G$1.TEST; no longer C5.1, C6.1, J6.SHIELD, R8.2
- net N$22: now also R27.2, U4G$1.AUTOEN_HS_SUSPD; no longer C16.1, FB3.2, J4.VBUS
- net N$23: now also R25.2, U4G$1.GANGED/SMBA2/HS_UP; no longer C10.1, FB1.2, J2.VBUS
- net N$24: now also R24.2, U4G$1.FPMGT/SMBA1/SS_UP; no longer C19.1, FB4.2, J5.VBUS
- net N$25: now also R22.2, R23.2, U4G$1.USB_VBUS; no longer R20.2, U6.ILIM
- net N$26: now also C27.1, U4G$1.USB_SSTXM_DN4; no longer C28.1, U$1G$2.GRSTZ
- net N$27: now also C26.1, U4G$1.USB_SSTXP_DN4; no longer R23.2, U$1G$2.USB_R1
- net N$28: now also C25.1, U4G$1.USB_SSTXM_DN3; no longer R17.2, U5.ILIM
- net N$29: now also C24.1, U4G$1.USB_SSTXP_DN3; no longer C29.1, R26.1, U$1G$2.XI, Y2.1
- net N$30: now also C23.1, U4G$1.USB_SSTXM_DN2; no longer C30.1, R26.2, U$1G$2.XO, Y2.2
- net N$31: now also C22.1, U4G$1.USB_SSTXP_DN2; no longer R25.2, U$1G$2.TEST
- net N$32: now also C21.1, U4G$1.USB_SSTXM_DN1; no longer C39.1, C40.1, C41.1, C42.1, C43.1, FB6.1, U$1G$3.VDD33_1, U$1G$3.VDD33_2, U$1G$3.VDD33_3, U$1G$3.VDD33_4
- net N$33: now also C20.1, U4G$1.USB_SSTXP_DN1; no longer R24.2, U$1G$2.AUTOENZ/HS_SUSPEND
- net N$35: now also C12.1, FB1.2, K2.VBUS; no longer C17.1, C18.1, J5.SHIELD, R12.2
- net N$36: now also C42.1, U5.SS; no longer C14.1, C15.1, J4.SHIELD, R11.2
- net N$38: now also C17.1, FB2.2; no longer C11.1, C12.1, J3.SHIELD, R9.2
- net N$9: now also R28.2, U4G$1.USB_R1; no longer R4.2, U$1G$4.FULLPWRMGMTZ/SMBA1
- net OVERCUR1Z: now also R39.1, U4G$1.OVERCURZ1; no longer R21.1, U$1G$1.OVERCUR1Z
- net OVERCUR2Z: now also R41.1, U4G$1.OVERCURZ2; no longer R22.1
- net OVERCUR3Z: now also R40.1, U4G$1.OVERCURZ3, U7.FAULT1Z; no longer R18.1, U5.FAULT1Z
- net OVERCUR4Z: now also R42.1, U4G$1.OVERCURZ4, U7.FAULT2Z; no longer R19.1, U5.FAULT2Z
- net USB_DM_DN1: now also K2.D-, U4G$1.USB_DM_DN1; no longer J2.D-, U$1G$1.USB_DM_DN1
- net USB_DM_DN2: now also K3.D-, U4G$1.USB_DM_DN2; no longer J3.D-
- net USB_DM_DN3: now also K4.D-, U4G$1.USB_DM_DN3; no longer J4.D-
- net USB_DM_DN4: now also K5.D-, U4G$1.USB_DM_DN4; no longer J5.D-
- net USB_DP_DN1: now also K2.D+, U4G$1.USB_DP_DN1; no longer J2.D+, U$1G$1.USB_DP_DN1
- net USB_DP_DN2: now also K3.D+, U4G$1.USB_DP_DN2; no longer J3.D+
- net USB_DP_DN3: now also K4.D+, U4G$1.USB_DP_DN3; no longer J4.D+
- net USB_DP_DN4: now also K5.D+, U4G$1.USB_DP_DN4; no longer J5.D+

Commit message: inital commit
Connections:
- removed net NSS_3P3V: U3.NSS
- new net NSS_3V3: U3.NSS, U8.PA7(PCINT7/ADC7/TOCC6/ICP1/TXD0/SS')
- net MISO_3V3: now also U8.PA5(PCINT5/ADC5/ACO0/TOCC4/T2/TXD1/MISO)
- net MOSI_3V3: now also U8.PA6(PCINT6/ADC6/ACO1/TOCC5/XCK1/SDA/MOSI)
- net SCK_3V3: now also U8.PA4(PCINT4/ADC4/AIN11/TOCC3/T1/RXD1/SCL/SCK)
Changed lines of the file:
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@@
 <?xml version="1.0" encoding="utf-8"?>
 <!DOCTYPE eagle SYSTEM "eagle.dtd">
-<eagle version="8.1.0">
+<eagle version="8.1.1">
 <drawing>
 <settings>
@@
 <net name="SCK_3V3" class="0">
 <segment>
-<wire x1="38.1" y1="7.62" x2="58.42" y2="7.62" width="0.1524" layer="91"/>
-<label x="58.42" y="7.62" size="1.778" layer="95" xref="yes"/>
-</segment>
-<segment>
 <pinref part="U3" gate="G$1" pin="SCK"/>
 <wire x1="-10.16" y1="63.5" x2="-12.7" y2="63.5" width="0.1524" layer="91"/>
 <label x="-12.7" y="63.5" size="1.778" layer="95" font="vector" rot="R180" xref="yes"/>
 </segment>
+<segment>
+<pinref part="U8" gate="G$1" pin="PA4(PCINT4/ADC4/AIN11/TOCC3/T1/RXD1/SCL/SCK)"/>
+<wire x1="38.1" y1="7.62" x2="48.26" y2="7.62" width="0.1524" layer="91"/>
+<label x="48.26" y="7.62" size="1.778" layer="95" xref="yes"/>
+</segment>
 </net>
 <net name="MISO_3V3" class="0">
-<segment>
-<wire x1="38.1" y1="2.54" x2="45.72" y2="2.54" width="0.1524" layer="91"/>
-<label x="45.72" y="2.54" size="1.778" layer="95" xref="yes"/>
-</segment>
 <segment>
 <pinref part="U3" gate="G$1" pin="MISO"/>
@@
 <label x="-12.7" y="68.58" size="1.778" layer="95" font="vector" rot="R180" xref="yes"/>
 </segment>
+<segment>
+<pinref part="U8" gate="G$1" pin="PA5(PCINT5/ADC5/ACO0/TOCC4/T2/TXD1/MISO)"/>
+<wire x1="38.1" y1="2.54" x2="48.26" y2="2.54" width="0.1524" layer="91"/>
+<label x="48.26" y="2.54" size="1.778" layer="95" xref="yes"/>
+</segment>
 </net>
 <net name="MOSI_3V3" class="0">
-<segment>
-<wire x1="38.1" y1="-2.54" x2="45.72" y2="-2.54" width="0.1524" layer="91"/>
-<label x="45.72" y="-2.54" size="1.778" layer="95" xref="yes"/>
-</segment>
 <segment>
 <pinref part="U3" gate="G$1" pin="MOSI"/>
@@
 <label x="-30.48" y="66.04" size="1.778" layer="95" font="vector" rot="R180" xref="yes"/>
 </segment>
-</net>
-<net name="NSS_3V3" class="0">
-<segment>
-<wire x1="38.1" y1="-7.62" x2="45.72" y2="-7.62" width="0.1524" layer="91"/>
-<label x="45.72" y="-7.62" size="1.778" layer="95" xref="yes"/>
+<segment>
+<pinref part="U8" gate="G$1" pin="PA6(PCINT6/ADC6/ACO1/TOCC5/XCK1/SDA/MOSI)"/>
+<wire x1="38.1" y1="-2.54" x2="48.26" y2="-2.54" width="0.1524" layer="91"/>
+<label x="48.26" y="-2.54" size="1.778" layer="95" xref="yes"/>
 </segment>
 </net>
@@
 </segment>
 </net>
-<net name="NSS_3P3V" class="0">
-<segment>
-<pinref part="U3" gate="G$1" pin="NSS"/>
-<wire x1="-10.16" y1="60.96" x2="-30.48" y2="60.96" width="0.1524" layer="91"/>
-<label x="-30.48" y="60.96" size="1.778" layer="95" font="vector" rot="R180" xref="yes"/>
-</segment>
-</net>
 <net name="DIO0_3V3" class="0">
 <segment>
@@
 </segment>
 </net>
+<net name="NSS_3V3" class="0">
+<segment>
+<pinref part="U8" gate="G$1" pin="PA7(PCINT7/ADC7/TOCC6/ICP1/TXD0/SS')"/>
+<wire x1="38.1" y1="-7.62" x2="48.26" y2="-7.62" width="0.1524" layer="91"/>
+<label x="48.26" y="-7.62" size="1.778" layer="95" xref="yes"/>
+</segment>
+<segment>
+<pinref part="U3" gate="G$1" pin="NSS"/>
+<wire x1="-10.16" y1="60.96" x2="-30.48" y2="60.96" width="0.1524" layer="91"/>
+<label x="-30.48" y="60.96" size="1.778" layer="95" font="vector" rot="R180" xref="yes"/>
+</segment>
+</net>

Commit message: 05/01/2017
Parts:
- C10, C16, C19, C33, C5: device SparkFun-Capacitors:1.0NF/1000PF-0603-50V-10% -> rcl:C-USC0603
- C11: device SparkFun-Capacitors:1.0UF-0603-16V-10% -> rcl:C-USC0603
- C12, C13, C17, C18, C20, C21, C22, C23, C24, C25, C26, C27, C28, C29, C31, C32, C35, C36, C37, C38, C39, C40, C41, C44, C45, C46, C47, C48, C49, C51, C52, C55, C56, C6, C8, C9: device SparkFun-Capacitors:0.1UF-0603-25V-(+80/-20%) -> rcl:C-USC0603
- C14, C15: device SparkFun-Capacitors:18PF-0603-50V-5% -> rcl:C-USC0603
- C30, C50, C7: device SparkFun-Capacitors:10UF-0603-6.3V-20% -> rcl:C-USC0603
- C34, C43: device SparkFun-Capacitors:4.7UF0603 -> rcl:C-USC0603
- C42: device SparkFun-Capacitors:10NF-0603-50V-10% -> rcl:C-USC0603
- R20, R21, R26, R30, R31, R36: device SparkFun-Resistors:1MOHM-0603-1/4W-5% -> rcl:R-US_R0603
- R22: device SparkFun-Resistors:100KOHM-0603-1/10W-1% -> rcl:R-US_R0603
- R23, R39, R40, R41, R42: device SparkFun-Resistors:10KOHM-0603-1/10W-1% -> rcl:R-US_R0603
- R24, R25, R27, R29, R32, R33, R34, R35: device SparkFun-Resistors:4.7KOHM-0603-1/10W-1% -> rcl:R-US_R0603
- R28: device SparkFun-Resistors:9.76KOHM-0603-1/10W-1% -> rcl:R-US_R0603
- R37, R38: device SparkFun-Resistors:26.7KOHM0603-1/10W-1% -> rcl:R-US_R0603
Connections:
- removed net N$45: C56.1, C58.+, U7.OUT2
- net +3V3_HUB: now also U4G$2.VDD33_1, U4G$2.VDD33_2, U4G$2.VDD33_3, U4G$2.VDD33_4
- net DN4_VBUS: now also C56.1, C58.+, U7.OUT2
- net GND: now also K4.GND_DRAIN, K5.GND_DRAIN; no longer U4G$2.VDD33_1, U4G$2.VDD33_2, U4G$2.VDD33_3, U4G$2.VDD33_4
- net N$38: now also K3.VBUS
Other:
- moved on the sheet: C10, C11, C12, C13, C14, C15, C16, C17, C18, C19, C20, C21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

Commit message: cinco de mayo
Parts:
- added C62: 4.7uF, rcl:C-USC0603
- added C63: 1.0uF, rcl:C-USC0603
- C20, C21, C22, C23, C24, C25, C26, C27, C8, C9: device rcl:C-USC0603 -> rcl:C-USC0402
Connections:
- net 3.3V: now also C63.1, IMU.2; no longer ENCODER.2
- net 5V: now also C62.1, ENCODER.1; no longer IMU.1
- net ACHANNEL_5V: now also ENCODER.2; no longer IMU.2
- net BCHANNEL_5V: now also ENCODER.4; no longer IMU.4
- net GND: now also C62.2, C63.2, ENCODER.3, IMU.1, U3.RESET; no longer ENCODER.1, IMU.3
- net I2C0_SCL: now also IMU.4; no longer ENCODER.4
- net I2C0_SDA: now also IMU.3; no longer ENCODER.3
- net N$26: now also U4G$1.USB_SSTXP_DN4; no longer U4G$1.USB_SSTXM_DN4
- net N$27: now also U4G$1.USB_SSTXM_DN4; no longer U4G$1.USB_SSTXP_DN4
- net N$28: now also U4G$1.USB_SSTXP_DN3; no longer U4G$1.USB_SSTXM_DN3
- net N$29: now also U4G$1.USB_SSTXM_DN3; no longer U4G$1.USB_SSTXP_DN3
- net N$30: now also U4G$1.USB_SSTXP_DN2; no longer U4G$1.USB_SSTXM_DN2
- net N$31: now also U4G$1.USB_SSTXM_DN2; no longer U4G$1.USB_SSTXP_DN2
- net N$32: now also U4G$1.USB_SSTXP_DN1; no longer U4G$1.USB_SSTXM_DN1
- net N$33: now also U4G$1.USB_SSTXM_DN1; no longer U4G$1.USB_SSTXP_DN1
Other:
- moved on the sheet: ENCODER, IMU
